File: _saved_comp2dvi2.sch (KiCad schematic (older format))
At the start: 30 parts, among them J1 Conn_Coaxial, J2 Conn_Coaxial, J3 Conn_Coaxial, J4 USB_B_Micro, J5 DVI-I-R, SW1 SW_DIP_x02, SW2 SW_DPDT_x2, U1 THS7368

Commit message: Bypass Cap Routing
Fixed routing so that the power from the USB goes to the 100nF bypass cap before hitting the chip. Thanks to Tianfeng for pointing this out. Gerbers updated as well.
Parts:
- J5: symbol SCART_to_DVI-A_Compact-eagle-import:DVI-I-R -> comp2dvi2-rescue:DVI-I-R-SCART_to_DVI-A_Compact-eagle-import
- SW2: symbol Switch2:SW_DPDT_x2 -> comp2dvi2-rescue:SW_DPDT_x2-Switch2
- U1: symbol THS7368:THS7368 -> comp2dvi2-rescue:THS7368-THS7368
Changed lines of the file:
@@
 $EndDescr
 $Comp
-L THS7368:THS7368 U1
+L comp2dvi2-rescue:THS7368-THS7368 U1
 U 1 1 5C9672D2
 P 5350 4500
@@
 Pb_OUT
 $Comp
-L SCART_to_DVI-A_Compact-eagle-import:DVI-I-R J5
+L comp2dvi2-rescue:DVI-I-R-SCART_to_DVI-A_Compact-eagle-import J5
 U 1 1 5C96A17A
 P 8550 3750
@@
 $EndComp
 $Comp
-L Switch2:SW_DPDT_x2 SW2
+L comp2dvi2-rescue:SW_DPDT_x2-Switch2 SW2
 U 1 1 5CB6A3DC
 P 6200 5700
